File: PCB/EagleV1/EagleV1.kicad_pcb (KiCad board)
At the start: 2 copper layers, 3.6 x 3.3 mm, 200 parts, among them J1 USB_C_Receptacle_USB2.0_16P, J2 USB_C_Receptacle_USB2.0_16P, J3 USB_C_Receptacle_USB2.0_16P, J4 USB_C_Receptacle_USB2.0_16P, SW1 SW_Push, SW10 SW_Push, SW11 SW_Push, SW12 SW_Push, SW13 SW_Push, SW14 SW_Push, SW15 SW_Push, SW16 SW_Push, SW17 SW_Push, SW18 SW_Push, SW19 SW_Push, SW2 SW_Push, SW20 SW_Push, SW21 SW_Push, SW22 SW_Push, SW23 SW_Push, SW24 SW_Push, SW25 SW_Push, SW26 SW_Push, SW27 SW_Push, SW28 SW_Push, SW29 SW_Push, SW3 SW_Push, SW30 SW_Push, SW31 SW_Push, SW32 SW_Push, SW33 SW_Push, SW34 SW_Push, SW35 SW_Push, SW36 SW_Push, SW37 SW_Push, SW38 SW_Push, SW39 SW_Push, SW4 SW_Push, SW40 SW_Push, SW41 SW_Push, SW42 SW_Push, SW5 SW_Push, SW6 SW_Push, SW7 SW_Push, SW8 SW_Push, SW9 SW_Push, SW98 TS-1088-AR02016, SW99 TS-1088-AR02016, U1 RP2040, U10 TLV1117-33, U11 USBLC6-2SC6, U12 SN74LVC1T45DCK, U2 TLV1117-33, U3 W25Q128JVS, U4 USBLC6-2SC6, U5 USBLC6-2SC6, U6 SN74LVC1T45DCK, U7 W25Q128JVS, U8 USBLC6-2SC6, U9 RP2040, Y1 Crystal_GND24, Y2 Crystal_GNDB24

Commit message: started keyboard rounting
Parts:
- C1, C10, C11, C12, C13, C14, C15, C16, C17, C18, C19, C2, C24, C25, C26, C27, C28, C29, C3, C30, C31, C32, C33, C34, C35, C36, C37, C38, C39, C4, C40, C41, C42, C43, C44, C45, C46, C47, C48, C49, C5, C50, C51, C52, C53, C54, C55, C56, C57, C58, C6, C7, C78, C8, C9, D1, D2, J1, J2, J3, J4, LED1, LED10, LED11, LED12, LED13, LED14, LED15, LED16, LED17, LED18, LED19, LED2, LED20, LED21, LED22, LED42, LED7, LED8, LED9, R1, R10, R11, R12, R13, R14, R15, R16, R2, R3, R4, R5, R6, R7, R8, R9, SW98, SW99, U1, U10, U11, U12, U2, U3, U4, U5, U6, U7, U8, U9, Y1, Y2: moved to B.Cu
- C20: renamed from C22; moved to B.Cu
- C21: renamed from C23; moved to B.Cu
- C22: renamed from C20; moved to B.Cu
- C23: renamed from C21; moved to B.Cu
- C59: renamed from C61; moved to B.Cu
- C60: renamed from C64; moved to B.Cu
- C61: renamed from C67; moved to B.Cu
- C62: renamed from C71; moved to B.Cu
- C63: renamed from C75; moved to B.Cu
- C64: renamed from C59; moved to B.Cu
- C65: renamed from C62; moved to B.Cu
- C66: renamed from C65; moved to B.Cu
- C67: renamed from C68; moved to B.Cu
- C68: renamed from C72; moved to B.Cu
- C69: renamed from C76; moved to B.Cu
- C70: renamed from C60; moved to B.Cu
- C71: renamed from C63; moved to B.Cu
- C72: renamed from C66; moved to B.Cu
- C73: renamed from C69; moved to B.Cu
- C74: renamed from C73; moved to B.Cu
- C75: renamed from C77; moved to B.Cu
- C76: renamed from C70; moved to B.Cu
- C77: renamed from C74; moved to B.Cu
- LED23: renamed from LED25; moved to B.Cu
- LED24: renamed from LED28; moved to B.Cu
- LED25: renamed from LED31; moved to B.Cu
- LED26: renamed from LED35; moved to B.Cu
- LED27: renamed from LED39; moved to B.Cu
- LED28: renamed from LED23; moved to B.Cu
- LED29: renamed from LED26; moved to B.Cu
- LED3: renamed from LED5; moved to B.Cu
- LED30: renamed from LED29; moved to B.Cu
- LED31: renamed from LED32; moved to B.Cu
- LED32: renamed from LED36; moved to B.Cu
- LED33: renamed from LED40; moved to B.Cu
- LED34: renamed from LED24; moved to B.Cu
- LED35: renamed from LED27; moved to B.Cu
- LED36: renamed from LED30; moved to B.Cu
- LED37: renamed from LED33; moved to B.Cu
- LED38: renamed from LED37; moved to B.Cu
- LED39: renamed from LED41; moved to B.Cu
- LED4: renamed from LED6; moved to B.Cu
- LED40: renamed from LED34; moved to B.Cu
- LED41: renamed from LED38; moved to B.Cu
- LED5: renamed from LED3; moved to B.Cu
- LED6: renamed from LED4; moved to B.Cu
- moved LED39 424.3 mm to (342.9, 120.6)
- moved R10 423.9 mm to (343.4, 172.9), turned to 180 degrees
- moved R11 423.9 mm to (343.4, 174.9), turned to 180 degrees
- moved R12 423.9 mm to (343.4, 176.8), turned to 180 degrees
- moved R13 423.9 mm to (343.4, 178.8), turned to 180 degrees
- moved R14 423.9 mm to (343.4, 180.8), turned to 180 degrees
- moved R15 423.9 mm to (343.4, 182.8), turned to 180 degrees
- moved R16 423.9 mm to (343.4, 184.8), turned to 180 degrees
- moved R9 423.9 mm to (343.4, 170.9), turned to 180 degrees
- moved LED27 423.8 mm to (342.9, 82.5)
- moved LED33 423.8 mm to (342.9, 101.6), turned to 180 degrees
- moved LED26 414.6 mm to (323.9, 80.6)
- moved LED32 413.9 mm to (323.9, 99.7), turned to 180 degrees
- moved LED38 413.6 mm to (323.9, 118.7)
- moved R3 404.4 mm to (220.0, 1.76), turned to 180 degrees
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Connections:
- net Net-(D1-A) renamed /LeftSide/VBUS
- net Net-(D2-A) renamed /RightSide/VBUSB
- net Net-(J1-CC1) renamed /LeftSide/CC1
- net Net-(J1-CC2) renamed /LeftSide/CC2
- net Net-(J3-CC1) renamed /RightSide/CC1B
- net Net-(J3-CC2) renamed /RightSide/CC2B
- net Net-(LED10-DIN) renamed LED10IN
- net Net-(LED10-DOUT) renamed LED11IN
- net Net-(LED11-DOUT) renamed LED12IN
- net Net-(LED19-DOUT) renamed LED20IN
- net Net-(LED20-DOUT) renamed LED21IN
- net Net-(LED7-DOUT) renamed LED8IN
- net Net-(LED8-DOUT) renamed LED9IN
- LED1 pad 2: Net-(LED1-DOUT) -> LED7IN
- LED1 pad 3: LED_5_data -> LED1IN
- LED12 pad 2: Net-(LED12-DOUT) -> LED18IN
- LED13 pad 2: Net-(LED13-DOUT) -> LED19IN
- LED13 pad 3: Net-(LED12-DOUT) -> LED13IN
- LED14 pad 2: Net-(LED14-DOUT) -> LED13IN
- LED14 pad 3: Net-(LED13-DOUT) -> LED14IN
- LED15 pad 2: Net-(LED15-DOUT) -> LED14IN
- LED15 pad 3: Net-(LED14-DOUT) -> LED15IN
- LED16 pad 2: Net-(LED16-DOUT) -> LED15IN
- LED16 pad 3: Net-(LED15-DOUT) -> LED16IN
- LED17 pad 2: Net-(LED17-DOUT) -> LED16IN
- LED17 pad 3: Net-(LED16-DOUT) -> LED17IN
- LED18 pad 2: Net-(LED18-DOUT) -> LED17IN
- LED18 pad 3: Net-(LED17-DOUT) -> LED18IN
- LED19 pad 3: Net-(LED18-DOUT) -> LED19IN
- LED2 pad 2: Net-(LED2-DOUT) -> LED1IN
- LED2 pad 3: Net-(LED1-DOUT) -> LED2IN
- LED3 pad 2: Net-(LED5-DOUT) -> LED2IN
- LED3 pad 3: Net-(LED2-DOUT) -> LED3IN
- LED4 pad 2: Net-(LED3-DIN) -> LED3IN
- LED4 pad 3: Net-(LED5-DOUT) -> LED4IN
- LED5 pad 2: Net-(LED3-DOUT) -> LED4IN
- LED5 pad 3: Net-(LED3-DIN) -> LED5IN
- LED6 pad 2: Net-(LED4-DOUT) -> LED5IN
- LED6 pad 3: Net-(LED3-DOUT) -> LED_5_data
- LED7 pad 3: Net-(LED4-DOUT) -> LED7IN
- R12 pad 1: QSPI_NCS -> QSPI_NCS_B_B
- R9 pad 2: QSPI_NCS -> QSPI_NCS_B_B
- U7 pad 1: QSPI_NCS -> QSPI_NCS_B_B
- U7 pad 2: QSPI_D1 -> QSPI_D1_B
- U7 pad 3: QSPI_D2 -> QSPI_D2_B
- U7 pad 5: QSPI_D0 -> QSPI_D0_B
- U7 pad 6: QSPI_CLK -> QSPI_CLK_B
- U7 pad 7: QSPI_D3 -> QSPI_D3_B
- U9 pad 51: QSPI_D3 -> QSPI_D3_B
- U9 pad 52: QSPI_CLK -> QSPI_CLK_B
- U9 pad 53: QSPI_D0 -> QSPI_D0_B
- U9 pad 54: QSPI_D2 -> QSPI_D2_B
- U9 pad 55: QSPI_D1 -> QSPI_D1_B
- U9 pad 56: QSPI_NCS -> QSPI_NCS_B
Routing:
- net +5V: track 0.00 -> 552.7 mm, vias 0 -> 10
- net SW1: track 0.00 -> 122.8 mm
- net SW7: track 0.00 -> 116.3 mm
- net SW2: track 0.00 -> 113.7 mm
- net SW13: track 0.00 -> 112.7 mm
- net SW8: track 0.00 -> 99.5 mm
- net SW14: track 0.00 -> 93.0 mm
- net SW3: track 0.00 -> 87.9 mm
- net LED19IN: track 0.00 -> 79.7 mm
- net SW9: track 0.00 -> 75.9 mm
- net SW15: track 0.00 -> 70.0 mm
- net SW4: track 0.00 -> 61.1 mm
- net SW10: track 0.00 -> 55.3 mm
- net SW19: track 0.00 -> 52.7 mm
- net SW16: track 0.00 -> 49.0 mm
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Other:
- board size 3.6 x 3.3 mm -> 285.8 x 103.7 mm
