File: PCB/EagleV1/EagleV1.kicad_pcb (KiCad board)
At the start: 2 copper layers, 285.8 x 103.7 mm, 204 parts, among them J1 USB_C_Receptacle_USB2.0_16P, J2 USB_C_Receptacle_USB2.0_16P, J3 USB_C_Receptacle_USB2.0_16P, J4 USB_C_Receptacle_USB2.0_16P, SW1 SW_Push, SW10 SW_Push, SW11 SW_Push, SW12 SW_Push, SW13 SW_Push, SW14 SW_Push, SW15 SW_Push, SW16 SW_Push, SW17 SW_Push, SW18 SW_Push, SW19 SW_Push, SW2 SW_Push, SW20 SW_Push, SW21 SW_Push, SW22 SW_Push, SW23 SW_Push, SW24 SW_Push, SW25 SW_Push, SW26 SW_Push, SW27 SW_Push, SW28 SW_Push, SW29 SW_Push, SW3 SW_Push, SW30 SW_Push, SW31 SW_Push, SW32 SW_Push, SW33 SW_Push, SW34 SW_Push, SW35 SW_Push, SW36 SW_Push, SW37 SW_Push, SW38 SW_Push, SW39 SW_Push, SW4 SW_Push, SW40 SW_Push, SW41 SW_Push, SW42 SW_Push, SW5 SW_Push, SW6 SW_Push, SW7 SW_Push, SW8 SW_Push, SW9 SW_Push, SW98 TS-1088-AR02016, SW99 TS-1088-AR02016, U1 RP2040, U10 TLV1117-33, U11 USBLC6-2SC6, U12 SN74LVC1T45DCK, U2 TLV1117-33, U3 W25Q128JVS, U4 USBLC6-2SC6, U5 USBLC6-2SC6, U6 SN74LVC1T45DCK, U7 W25Q128JVS, U8 USBLC6-2SC6, U9 RP2040, Y1 Crystal_GND24, Y2 Crystal_GNDB24

Commit message: routed all the tracks and smds
Parts:
- moved R13 158.1 mm to (226.9, 72.0), turned to -90 degrees
- moved R16 156.4 mm to (237.5, 69.7), turned to -90 degrees
- moved R14 155.6 mm to (232.2, 72.0), turned to -90 degrees
- moved R12 147.4 mm to (236.0, 75.9)
- moved C45 143.0 mm to (223.1, 80.4)
- moved R11 141.9 mm to (230.0, 85.7), turned to -90 degrees
- moved R9 141.7 mm to (238.2, 75.9)
- moved C49 140.5 mm to (220.8, 92.1)
- moved R10 139.9 mm to (231.0, 85.7), turned to -90 degrees
- moved C47 137.8 mm to (227.1, 86.2), turned to 90 degrees
- moved R15 137.7 mm to (234.2, 98.9), turned to 0 degrees
- moved U10 135.4 mm to (221.6, 86.2), turned to -90 degrees
- moved C42 133.3 mm to (228.7, 86.2), turned to 90 degrees
- moved C43 132.5 mm to (226.7, 73.8), turned to 0 degrees
- moved U9 129.7 mm to (231.7, 92.7)
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- renumbered SW98 to RESET
Connections:
- net Net-(LED22-DOUT) renamed LED23IN
- net Net-(LED23-DOUT) renamed LED24IN
- net Net-(LED24-DOUT) renamed LED25IN
- net Net-(LED25-DOUT) renamed LED26IN
- net Net-(LED26-DOUT) renamed LED27IN
- net Net-(LED34-DOUT) renamed LED35IN
- net Net-(LED35-DOUT) renamed LED36IN
- net Net-(LED36-DOUT) renamed LED37IN
- net Net-(LED37-DOUT) renamed LED38IN
- net Net-(LED38-DOUT) renamed LED39IN
- net Net-(R9-Pad1) renamed /RightSide/NCSB
- C58 pad 1: GNDB -> GND
- C58 pad 2: +5VB -> +5V
- C59 pad 1: GNDB -> GND
- C59 pad 2: +5VB -> +5V
- C60 pad 1: GNDB -> GND
- C60 pad 2: +5VB -> +5V
- C61 pad 1: GNDB -> GND
- C61 pad 2: +5VB -> +5V
- C62 pad 1: GNDB -> GND
- C62 pad 2: +5VB -> +5V
- C63 pad 1: GNDB -> GND
- C63 pad 2: +5VB -> +5V
- C64 pad 1: GNDB -> GND
- C64 pad 2: +5VB -> +5V
- C65 pad 1: GNDB -> GND
- C65 pad 2: +5VB -> +5V
- C66 pad 1: GNDB -> GND
- C66 pad 2: +5VB -> +5V
- C67 pad 1: GNDB -> GND
- C67 pad 2: +5VB -> +5V
- C68 pad 1: GNDB -> GND
- C68 pad 2: +5VB -> +5V
- C69 pad 1: GNDB -> GND
- C69 pad 2: +5VB -> +5V
- C70 pad 1: GNDB -> GND
- C70 pad 2: +5VB -> +5V
- C71 pad 1: GNDB -> GND
- C71 pad 2: +5VB -> +5V
- C72 pad 1: GNDB -> GND
- C72 pad 2: +5VB -> +5V
- C73 pad 1: GNDB -> GND
- C73 pad 2: +5VB -> +5V
- C74 pad 1: GNDB -> GND
- C74 pad 2: +5VB -> +5V
- C75 pad 1: GNDB -> GND
- C75 pad 2: +5VB -> +5V
- C76 pad 1: GNDB -> GND
- C76 pad 2: +5VB -> +5V
- C77 pad 1: GNDB -> GND
- C77 pad 2: +5VB -> +5V
- C78 pad 1: GNDB -> GND
- C78 pad 2: +5VB -> +5V
- LED22 pad 1: +5VB -> +5V
- LED22 pad 4: GNDB -> GND
- LED23 pad 1: +5VB -> +5V
- LED23 pad 4: GNDB -> GND
- LED24 pad 1: +5VB -> +5V
- LED24 pad 4: GNDB -> GND
- LED25 pad 1: +5VB -> +5V
- LED25 pad 4: GNDB -> GND
- LED26 pad 1: +5VB -> +5V
- LED26 pad 4: GNDB -> GND
- LED27 pad 1: +5VB -> +5V
- LED27 pad 2: Net-(LED27-DOUT) -> LED33IN
- LED27 pad 4: GNDB -> GND
- LED28 pad 1: +5VB -> +5V
- LED28 pad 2: Net-(LED28-DOUT) -> LED34IN
- LED28 pad 3: Net-(LED27-DOUT) -> LED28IN
- LED28 pad 4: GNDB -> GND
- LED29 pad 1: +5VB -> +5V
- LED29 pad 2: Net-(LED29-DOUT) -> LED28IN
- LED29 pad 3: Net-(LED28-DOUT) -> LED29IN
- LED29 pad 4: GNDB -> GND
- LED30 pad 1: +5VB -> +5V
- LED30 pad 2: Net-(LED30-DOUT) -> LED29IN
- LED30 pad 3: Net-(LED29-DOUT) -> LED30IN
- LED30 pad 4: GNDB -> GND
- LED31 pad 1: +5VB -> +5V
- LED31 pad 2: Net-(LED31-DOUT) -> LED30IN
- LED31 pad 3: Net-(LED30-DOUT) -> LED31IN
- LED31 pad 4: GNDB -> GND
- LED32 pad 1: +5VB -> +5V
- LED32 pad 2: Net-(LED32-DOUT) -> LED31IN
- LED32 pad 3: Net-(LED31-DOUT) -> LED32IN
- LED32 pad 4: GNDB -> GND
- LED33 pad 1: +5VB -> +5V
- LED33 pad 2: Net-(LED33-DOUT) -> LED32IN
- LED33 pad 3: Net-(LED32-DOUT) -> LED33IN
- LED33 pad 4: GNDB -> GND
- LED34 pad 1: +5VB -> +5V
- LED34 pad 3: Net-(LED33-DOUT) -> LED34IN
- LED34 pad 4: GNDB -> GND
- LED35 pad 1: +5VB -> +5V
- LED35 pad 4: GNDB -> GND
- LED36 pad 1: +5VB -> +5V
- LED36 pad 4: GNDB -> GND
- LED37 pad 1: +5VB -> +5V
- LED37 pad 4: GNDB -> GND
- LED38 pad 1: +5VB -> +5V
- LED38 pad 4: GNDB -> GND
- LED39 pad 1: +5VB -> +5V
- LED39 pad 2: Net-(LED39-DOUT) -> LED42IN
- LED39 pad 4: GNDB -> GND
- LED40 pad 1: +5VB -> +5V
- LED40 pad 2: Net-(LED40-DOUT) -> unconnected-(LED40-DOUT-Pad2)
- LED40 pad 3: Net-(LED39-DOUT) -> LED40IN
- LED40 pad 4: GNDB -> GND
- LED41 pad 1: +5VB -> +5V
- LED41 pad 2: Net-(LED41-DOUT) -> LED40IN
- LED41 pad 3: Net-(LED40-DOUT) -> LED41IN
- LED41 pad 4: GNDB -> GND
- LED42 pad 1: +5VB -> +5V
- LED42 pad 2: unconnected-(LED42-DOUT-Pad2) -> LED41IN
- LED42 pad 3: Net-(LED41-DOUT) -> LED42IN
- LED42 pad 4: GNDB -> GND
- R12 pad 1: QSPI_NCS_B_B -> QSPI_NCS_B
- R9 pad 2: QSPI_NCS_B_B -> QSPI_NCS_B
- U7 pad 1: QSPI_NCS_B_B -> QSPI_NCS_B
- U9 pad 11: unconnected-(U9-GPIO8-Pad11) -> SW27
- U9 pad 12: unconnected-(U9-GPIO9-Pad12) -> SW28
- U9 pad 13: unconnected-(U9-GPIO10-Pad13) -> SW29
- U9 pad 14: unconnected-(U9-GPIO11-Pad14) -> SW30
- U9 pad 15: unconnected-(U9-GPIO12-Pad15) -> SW31
- U9 pad 16: unconnected-(U9-GPIO13-Pad16) -> SW32
- U9 pad 17: unconnected-(U9-GPIO14-Pad17) -> SW33
- U9 pad 27: unconnected-(U9-GPIO16-Pad27) -> SW34
- U9 pad 28: unconnected-(U9-GPIO17-Pad28) -> SW35
- U9 pad 29: unconnected-(U9-GPIO18-Pad29) -> SW36
- U9 pad 30: unconnected-(U9-GPIO19-Pad30) -> SW37
- U9 pad 31: unconnected-(U9-GPIO20-Pad31) -> SW38
- U9 pad 32: unconnected-(U9-GPIO21-Pad32) -> SW39
- U9 pad 34: unconnected-(U9-GPIO22-Pad34) -> SW42
- U9 pad 35: unconnected-(U9-GPIO23-Pad35) -> SW41
- U9 pad 36: unconnected-(U9-GPIO24-Pad36) -> SW40
- U9 pad 5: unconnected-(U9-GPIO3-Pad5) -> SW22
- U9 pad 6: unconnected-(U9-GPIO4-Pad6) -> SW23
- U9 pad 7: unconnected-(U9-GPIO5-Pad7) -> SW24
- U9 pad 8: unconnected-(U9-GPIO6-Pad8) -> SW25
- U9 pad 9: unconnected-(U9-GPIO7-Pad9) -> SW26
Routing:
- net +5V: track 639.1 -> 1184.6 mm, vias 14 -> 19
- net SW39: track 0.00 -> 140.8 mm
- net SW27: track 0.00 -> 134.3 mm
- net SW33: track 0.00 -> 123.8 mm
- net SW38: track 0.00 -> 117.7 mm
- net SW26: track 0.00 -> 113.6 mm
- net +5VB: track 0.00 -> 103.1 mm, vias 0 -> 2
- net SW32: track 0.00 -> 102.3 mm
- net SW37: track 0.00 -> 91.2 mm
- net SW25: track 0.00 -> 88.9 mm
- net +3V3B: track 0.00 -> 88.4 mm, vias 0 -> 3
- net LED42IN: track 0.00 -> 84.1 mm
- net SW31: track 0.00 -> 77.0 mm
- net SW36: track 0.00 -> 68.6 mm
- net SW42: track 0.00 -> 68.4 mm
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- added copper zone on B.Cu, net +1V1B
- added copper zone on B.Cu, net +3V3B
- added copper zone on B.Cu, net /RightSide/VBUSB
- added copper zone on F.Cu, net D+
- added copper zone on F.Cu, net GND
- added copper zone on B.Cu, net GNDB
Other:
- board size 285.8 x 103.7 mm -> 285.2 x 103.7 mm

Commit message: Finished layout, both halves
Parts:
- renumbered RESET to SW98
Connections:
- C58 pad 1: GND -> GNDB
- C58 pad 2: +5V -> +5VB
- C59 pad 1: GND -> GNDB
- C59 pad 2: +5V -> +5VB
- C60 pad 1: GND -> GNDB
- C60 pad 2: +5V -> +5VB
- C61 pad 1: GND -> GNDB
- C61 pad 2: +5V -> +5VB
- C62 pad 1: GND -> GNDB
- C62 pad 2: +5V -> +5VB
- C63 pad 1: GND -> GNDB
- C63 pad 2: +5V -> +5VB
- C64 pad 1: GND -> GNDB
- C64 pad 2: +5V -> +5VB
- C65 pad 1: GND -> GNDB
- C65 pad 2: +5V -> +5VB
- C66 pad 1: GND -> GNDB
- C66 pad 2: +5V -> +5VB
- C67 pad 1: GND -> GNDB
- C67 pad 2: +5V -> +5VB
- C68 pad 1: GND -> GNDB
- C68 pad 2: +5V -> +5VB
- C69 pad 1: GND -> GNDB
- C69 pad 2: +5V -> +5VB
- C70 pad 1: GND -> GNDB
- C70 pad 2: +5V -> +5VB
- C71 pad 1: GND -> GNDB
- C71 pad 2: +5V -> +5VB
- C72 pad 1: GND -> GNDB
- C72 pad 2: +5V -> +5VB
- C73 pad 1: GND -> GNDB
- C73 pad 2: +5V -> +5VB
- C74 pad 1: GND -> GNDB
- C74 pad 2: +5V -> +5VB
- C75 pad 1: GND -> GNDB
- C75 pad 2: +5V -> +5VB
- C76 pad 1: GND -> GNDB
- C76 pad 2: +5V -> +5VB
- C77 pad 1: GND -> GNDB
- C77 pad 2: +5V -> +5VB
- C78 pad 1: GND -> GNDB
- C78 pad 2: +5V -> +5VB
- C81 pad 2: GND -> GNDB
- C82 pad 2: GND -> GNDB
- LED22 pad 1: +5V -> +5VB
- LED22 pad 4: GND -> GNDB
- LED23 pad 1: +5V -> +5VB
- LED23 pad 4: GND -> GNDB
- LED24 pad 1: +5V -> +5VB
- LED24 pad 4: GND -> GNDB
- LED25 pad 1: +5V -> +5VB
- LED25 pad 4: GND -> GNDB
- LED26 pad 1: +5V -> +5VB
- LED26 pad 4: GND -> GNDB
- LED27 pad 1: +5V -> +5VB
- LED27 pad 4: GND -> GNDB
- LED28 pad 1: +5V -> +5VB
- LED28 pad 4: GND -> GNDB
- LED29 pad 1: +5V -> +5VB
- LED29 pad 4: GND -> GNDB
- LED30 pad 1: +5V -> +5VB
- LED30 pad 4: GND -> GNDB
- LED31 pad 1: +5V -> +5VB
- LED31 pad 4: GND -> GNDB
- LED32 pad 1: +5V -> +5VB
- LED32 pad 4: GND -> GNDB
- LED33 pad 1: +5V -> +5VB
- LED33 pad 4: GND -> GNDB
- LED34 pad 1: +5V -> +5VB
- LED34 pad 4: GND -> GNDB
- LED35 pad 1: +5V -> +5VB
- LED35 pad 4: GND -> GNDB
- LED36 pad 1: +5V -> +5VB
- LED36 pad 4: GND -> GNDB
- LED37 pad 1: +5V -> +5VB
- LED37 pad 4: GND -> GNDB
- LED38 pad 1: +5V -> +5VB
- LED38 pad 4: GND -> GNDB
- LED39 pad 1: +5V -> +5VB
- LED39 pad 4: GND -> GNDB
- LED40 pad 1: +5V -> +5VB
- LED40 pad 4: GND -> GNDB
- LED41 pad 1: +5V -> +5VB
- LED41 pad 4: GND -> GNDB
- LED42 pad 1: +5V -> +5VB
- LED42 pad 4: GND -> GNDB
Routing:
- net +5VB: track 103.1 -> 657.5 mm, vias 2 -> 8
- net +5V: track 1184.6 -> 651.0 mm, vias 19 -> 15
- net GND: track 10.1 -> 68.4 mm, vias 4 -> 137
- net GNDB: track 10.1 -> 59.0 mm, vias 2 -> 138
- net /RightSide/DIR3V3B: track 0.00 -> 2.46 mm
- net SW1: track 150.5 -> 149.9 mm
- added copper zone on F.Cu, net GNDB
- removed copper zone on F.Cu, net D+
Other:
- board text added: "RESET"

Commit message: finished the PCB layout, exported gerbers
Parts:
- added Mousbites 0.5mm NPTH with 0.3mm spacing: Corne_mousebites, RandomStuff4Keebs:Corne_mousebites, F.Cu at (320.9, 66.6)
- added Mousbites 0.5mm NPTH with 0.3mm spacing: Corne_mousebites, RandomStuff4Keebs:Corne_mousebites, F.Cu at (307.2, 124.8)
- added Mousbites 0.5mm NPTH with 0.3mm spacing: Corne_mousebites, RandomStuff4Keebs:Corne_mousebites, F.Cu at (169.9, 62.8)
- added Mousbites 0.5mm NPTH with 0.3mm spacing: Corne_mousebites, RandomStuff4Keebs:Corne_mousebites, F.Cu at (242.0, 62.8)
- added Mousbites 0.5mm NPTH with 0.3mm spacing: Corne_mousebites, RandomStuff4Keebs:Corne_mousebites, F.Cu at (171.5, 62.8)
- added Mousbites 0.5mm NPTH with 0.3mm spacing: Corne_mousebites, RandomStuff4Keebs:Corne_mousebites, F.Cu at (108.7, 124.8)
- added Mousbites 0.5mm NPTH with 0.3mm spacing: Corne_mousebites, RandomStuff4Keebs:Corne_mousebites, F.Cu at (91.0, 66.6)
- added Mousbites 0.5mm NPTH with 0.3mm spacing: Corne_mousebites, RandomStuff4Keebs:Corne_mousebites, F.Cu at (339.3, 124.8)
- added Mousbites 0.5mm NPTH with 0.3mm spacing: Corne_mousebites, RandomStuff4Keebs:Corne_mousebites, F.Cu at (76.6, 124.8)
- added Mousbites 0.5mm NPTH with 0.3mm spacing: Corne_mousebites, RandomStuff4Keebs:Corne_mousebites, F.Cu at (322.5, 66.6)
- added Mousbites 0.5mm NPTH with 0.3mm spacing: Corne_mousebites, RandomStuff4Keebs:Corne_mousebites, F.Cu at (243.6, 62.8)
- added Mousbites 0.5mm NPTH with 0.3mm spacing: Corne_mousebites, RandomStuff4Keebs:Corne_mousebites, F.Cu at (92.6, 66.6)
- added REF**: M2SpacerHole3.2mm, RandomStuff4Keebs:M2SpacerHole3.2mm, F.Cu at (295.3, 75.6)
- added REF**: M2SpacerHole3.2mm, RandomStuff4Keebs:M2SpacerHole3.2mm, F.Cu at (333.4, 87.0)
- added REF**: M2SpacerHole3.2mm, RandomStuff4Keebs:M2SpacerHole3.2mm, F.Cu at (133.3, 109.5)
- added REF**: M2SpacerHole3.2mm, RandomStuff4Keebs:M2SpacerHole3.2mm, F.Cu at (257.2, 101.0)
- added REF**: M2SpacerHole3.2mm, RandomStuff4Keebs:M2SpacerHole3.2mm, F.Cu at (161.9, 83.9)
- added REF**: M2SpacerHole3.2mm, RandomStuff4Keebs:M2SpacerHole3.2mm, F.Cu at (85.7, 87.0)
- added REF**: M2SpacerHole3.2mm, RandomStuff4Keebs:M2SpacerHole3.2mm, F.Cu at (85.7, 106.1)
- added REF**: M2SpacerHole3.2mm, RandomStuff4Keebs:M2SpacerHole3.2mm, F.Cu at (257.2, 83.9)
- added REF**: M2SpacerHole3.2mm, RandomStuff4Keebs:M2SpacerHole3.2mm, F.Cu at (161.9, 102.9)
- added REF**: M2SpacerHole3.2mm, RandomStuff4Keebs:M2SpacerHole3.2mm, F.Cu at (333.4, 106.1)
- added REF**: M2SpacerHole3.2mm, RandomStuff4Keebs:M2SpacerHole3.2mm, F.Cu at (123.8, 75.6)
- added REF**: M2SpacerHole3.2mm, RandomStuff4Keebs:M2SpacerHole3.2mm, F.Cu at (285.8, 109.5)
Routing:
- net +5VB: track 657.5 -> 660.2 mm
- net SW11: track 83.5 -> 85.0 mm
- net SW7: track 145.2 -> 146.2 mm
- net +5V: track 651.0 -> 651.8 mm
Other:
- board size 285.2 x 103.7 mm -> 285.7 x 123.8 mm

Commit message: edited LED caps via placement and added some finishing touches
Parts:
- added G***: LOGO, RandomStuff4Keebs:cesky_lev, F.Cu at (287.0, 118.5)
- added G***: LOGO, RandomStuff4Keebs:cesky_lev, F.Cu at (132.1, 118.5)
- added REF**: my_sign, RandomStuff4Keebs:my_sign, F.Cu at (108.4, 124.4)
Routing:
- net GND: track 68.4 -> 62.5 mm
Other:
- board text added: "designed by Jan Kaucký"
