File: PCB/EagleV1/LeftSide.kicad_sch (KiCad schematic)
At the start: 48 parts, among them J1 USB_C_Receptacle_USB2.0_16P, SW1 SW_Push, SW10 SW_Push, SW11 SW_Push, SW12 SW_Push, SW13 SW_Push, SW14 SW_Push, SW15 SW_Push, SW16 SW_Push, SW17 SW_Push, SW18 SW_Push, SW19 SW_Push, SW2 SW_Push, SW20 SW_Push, SW21 SW_Push, SW22 TS-1088-AR02016, SW3 SW_Push, SW4 SW_Push, SW5 SW_Push, SW6 SW_Push, SW7 SW_Push, SW8 SW_Push, SW9 SW_Push, U1 RP2040, U2 AMS1117-3.3, U3 W25Q128JVS, U4 USBLC6-2SC6

Commit message: finished schematic
Parts:
- removed SW14, SW7: SW_Push, symbol Switch:SW_Push
- removed U2: AMS1117-3.3, Package_TO_SOT_SMD:SOT-223-3_TabPin2, symbol Regulator_Linear:AMS1117-3.3
- added C16, C17: 15p, Capacitor_SMD:C_0402_1005Metric, symbol Device:C
- added C18, C19, C20, C21, C22, C23, C24, C25, C26, C27, C28, C29, C30, C31, C32, C33, C34, C35, C36, C37, C38, C39: 100n, Capacitor_SMD:C_0402_1005Metric, symbol Device:C
- added D1: SS34, Diode_SMD:D_SMA, symbol Diode:SS34
- added J2: USB_C_Receptacle_USB2.0_16P, Connector_USB:USB_C_Receptacle_G-Switch_GT-USB-7010ASV, symbol Connector:USB_C_Receptacle_USB2.0_16P
- added LED1, LED10, LED11, LED12, LED13, LED14, LED15, LED16, LED17, LED18, LED19, LED2, LED20, LED21, LED3, LED4, LED5, LED6, LED7, LED8, LED9: SK6812MINI-E, PCM_marbastlib-various:LED_6028R, symbol PCM_marbastlib-various:SK6812MINI-E
- added R7: 1k, Resistor_SMD:R_0402_1005Metric, symbol Device:R
- added R8: 10k, Resistor_SMD:R_0402_1005Metric, symbol Device:R
- added SW17, SW18: SW_Push, RandomStuff4Keebs:SW_Redragon_LowProfile_PCB_1.00u, symbol Switch:SW_Push
- added U2: TLV1117-33, Package_TO_SOT_SMD:SOT-223-3_TabPin2, symbol Regulator_Linear:TLV1117-33
- added U5: USBLC6-2SC6, Package_TO_SOT_SMD:SOT-23-6, symbol Power_Protection:USBLC6-2SC6
- added U6: SN74LVC1T45DCK, Package_TO_SOT_SMD:SOT-363_SC-70-6, symbol Logic_LevelTranslator:SN74LVC1T45DCK
- added Y1: Crystal_GND24, Crystal:Crystal_SMD_3225-4Pin_3.2x2.5mm, symbol Device:Crystal_GND24
- C1, C2: value 10uF -> 1u
- C11, C9: footprint Capacitor_SMD:C_0402_1005Metric -> Capacitor_SMD:C_0603_1608Metric
- R5, R6: footprint (none) -> Resistor_SMD:R_0402_1005Metric
- SW1, SW19, SW2, SW20, SW21, SW3, SW4, SW5, SW6: footprint (none) -> RandomStuff4Keebs:SW_Redragon_LowProfile_PCB_1.00u
- SW10: renamed from SW11; footprint (none) -> RandomStuff4Keebs:SW_Redragon_LowProfile_PCB_1.00u
- SW11: renamed from SW12; footprint (none) -> RandomStuff4Keebs:SW_Redragon_LowProfile_PCB_1.00u
- SW12: renamed from SW13; footprint (none) -> RandomStuff4Keebs:SW_Redragon_LowProfile_PCB_1.00u
- SW13: renamed from SW15; footprint (none) -> RandomStuff4Keebs:SW_Redragon_LowProfile_PCB_1.00u
- SW14: renamed from SW16; footprint (none) -> RandomStuff4Keebs:SW_Redragon_LowProfile_PCB_1.00u
- SW15: renamed from SW17; footprint (none) -> RandomStuff4Keebs:SW_Redragon_LowProfile_PCB_1.00u
- SW16: renamed from SW18; footprint (none) -> RandomStuff4Keebs:SW_Redragon_LowProfile_PCB_1.00u
- SW7: renamed from SW8; footprint (none) -> RandomStuff4Keebs:SW_Redragon_LowProfile_PCB_1.00u
- SW8: renamed from SW9; footprint (none) -> RandomStuff4Keebs:SW_Redragon_LowProfile_PCB_1.00u
- SW9: renamed from SW10; footprint (none) -> RandomStuff4Keebs:SW_Redragon_LowProfile_PCB_1.00u
- renumbered SW22 to SW98
Connections:
- net +3.3V is gone; now on net +3V3: C2.1
- net +3V3: now also C10.1, C3.1, C4.1, C5.1, C6.1, C7.1, C8.1, C9.1, U1.1 (IOVDD), U1.10 (IOVDD), U1.22 (IOVDD), U1.26 (RUN), U1.33 (IOVDD), U1.42 (IOVDD), U1.43 (ADC_AVDD), U1.44 (VREG_IN), U1.48 (USB_VDD), U1.49 (IOVDD), R8.2, U2.2 (VO), U6.1 (VCCA)
- net +5V: now also C15.2, C18.2, C19.2, C20.2, C21.2, C22.2, C23.2, C24.2, C25.2, C26.2, C27.2, C28.2, C29.2, C30.2, C31.2, C32.2, C33.2, C34.2, C35.2, C36.2, C37.2, C38.2, C39.2, D1.1 (K), J2.A4 (VBUS), J2.A9 (VBUS), J2.B4 (VBUS), J2.B9 (VBUS), LED1.1 (VDD), LED10.1 (VDD), LED11.1 (VDD), LED12.1 (VDD), LED13.1 (VDD), LED14.1 (VDD), LED15.1 (VDD), LED16.1 (VDD), LED17.1 (VDD), LED18.1 (VDD), LED19.1 (VDD), LED2.1 (VDD), LED20.1 (VDD), LED21.1 (VDD), LED3.1 (VDD), LED4.1 (VDD), LED5.1 (VDD), LED6.1 (VDD), LED7.1 (VDD), LED8.1 (VDD), LED9.1 (VDD), U2.3 (VI), U5.5 (VBUS), U6.6 (VCCB); no longer C15.1, J1.A4 (VBUS), J1.A9 (VBUS), J1.B4 (VBUS), J1.B9 (VBUS)
- net GND: now also C15.1, SW1.2, SW10.2, SW11.2, SW12.2, SW13.2, SW14.2, SW15.2, SW16.2, SW19.2, SW2.2, SW20.2, SW21.2, SW3.2, SW4.2, SW5.2, SW6.2, SW7.2, SW8.2, SW9.2, U3.4 (GND), C16.2, C17.2, C18.1, C19.1, C20.1, C21.1, C22.1, C23.1, C24.1, C25.1, C26.1, C27.1, C28.1, C29.1, C30.1, C31.1, C32.1, C33.1, C34.1, C35.1, C36.1, C37.1, C38.1, C39.1, J2.A1 (GND), J2.A12 (GND), J2.B1 (GND), J2.B12 (GND), J2.S1 (SHIELD), LED1.4 (VSS), LED10.4 (VSS), LED11.4 (VSS), LED12.4 (VSS), LED13.4 (VSS), LED14.4 (VSS), LED15.4 (VSS), LED16.4 (VSS), LED17.4 (VSS), LED18.4 (VSS), LED19.4 (VSS), LED2.4 (VSS), LED20.4 (VSS), LED21.4 (VSS), LED3.4 (VSS), LED4.4 (VSS), LED5.4 (VSS), LED6.4 (VSS), LED7.4 (VSS), LED8.4 (VSS), LED9.4 (VSS), SW17.2, SW18.2, U2.1 (GND), U5.2 (GND), U6.2 (GND), Y1.2, Y1.4; no longer C15.2
- net SW3: now reaches SW3.1
- net SW3: now also U1.9 (GPIO7)
- net SW12: now reaches SW12.1
- net SW12: now also U1.27 (GPIO16)
- net SW19: now reaches SW19.1
- net SW19: now also U1.35 (GPIO23)
- net SW5: now reaches SW5.1
- net SW5: now also U1.12 (GPIO9)
- net +1V1: now reaches C11.1, C12.1, C13.1, U1.23 (DVDD), U1.45 (VREG_VOUT), U1.50 (DVDD)
- net SW11: now reaches SW11.1
- net SW11: now also U1.18 (GPIO15)
- net SW8: now reaches SW8.1
- net SW8: now also U1.15 (GPIO12)
- net SW16: now reaches SW16.1
- net SW16: now also U1.31 (GPIO20)
- net SW15: now reaches SW15.1
- net SW15: now also U1.30 (GPIO19)
- net SW7: now reaches SW7.1
- net SW7: now also U1.14 (GPIO11)
- net SW9: now reaches SW9.1
- net SW9: now also U1.16 (GPIO13)
- net SW10: now reaches SW10.1
- net SW10: now also U1.17 (GPIO14)
- net SW21: now reaches SW21.1
- net SW21: now also U1.37 (GPIO25)
- net D+: now reaches U4.6 (I/O1)
- net D+: now also J1.A6 (D+), J1.B6 (D+); no longer R4.1
- net D-: now reaches J1.A7 (D-), J1.B7 (D-)
- net D-: now also U4.4 (I/O2); no longer U4.1 (I/O1)
- net D_N: now reaches R3.1
- net D_N: now also U4.3 (I/O2); no longer U4.4 (I/O2)
- net SW14: now reaches SW14.1
- net SW14: now also U1.29 (GPIO18)
- net QSPI_NCS: now reaches R5.1, R6.2, U1.56 (QSPI_SS), U3.1 (~{CS})
- net QSPI_D1: now reaches U1.55 (QSPI_SD1), U3.2 (DO(IO1))
- net QSPI_D2: now reaches U1.54 (QSPI_SD2), U3.3 (IO2)
- net QSPI_D0: now reaches U1.53 (QSPI_SD0), U3.5 (DI(IO0))
- net QSPI_CLK: now reaches U1.52 (QSPI_SCLK), U3.6 (CLK)
- net QSPI_D3: now reaches U1.51 (QSPI_SD3), U3.7 (IO3)
- net SW6: now reaches SW6.1
- net SW6: now also U1.13 (GPIO10)
- net SW4: now reaches SW4.1
- net SW4: now also U1.11 (GPIO8)
- net SW20: now reaches SW20.1
- net SW20: now also U1.36 (GPIO24)
- net SW2: now reaches SW2.1
- net SW2: now also U1.8 (GPIO6)
- net SW13: now reaches SW13.1
- net SW13: now also U1.28 (GPIO17)
- net TX: now reaches U1.2 (GPIO0)
- net TX: now also U5.6 (I/O1)
- net XIN: now reaches U1.20 (XIN)
- net XIN: now also C17.1, Y1.3
- net XOUT: now reaches U1.21 (XOUT)
- net XOUT: now also R7.1
- net RX: now reaches U1.3 (GPIO1)
- net RX: now also U5.4 (I/O2)
- net SW17: now reaches U1.32 (GPIO21)
- net SW17: now also SW17.1
- net SW18: now reaches U1.34 (GPIO22)
- net SW18: now also SW18.1
- net LED_33_data: now reaches U1.4 (GPIO2)
- net LED_33_data: now also U6.3 (A)
- net SW1: now reaches U1.7 (GPIO5)
- net SW1: now also SW1.1
- new net: R8.1, U6.5 (DIR)
- new net: D1.2 (A), J1.A4 (VBUS), J1.A9 (VBUS), J1.B4 (VBUS), J1.B9 (VBUS)
- new net: LED18.2 (DOUT), LED19.3 (DIN)
- new net: LED17.2 (DOUT), LED18.3 (DIN)
- new net: LED20.2 (DOUT), LED21.3 (DIN)
- new net: LED16.2 (DOUT), LED17.3 (DIN)
- new net: J2.A7 (D-), J2.B7 (D-), U5.1 (I/O1)
- new net: J2.A6 (D+), J2.B6 (D+), U5.3 (I/O2)
- new net: C16.1, R7.2, Y1.1
- new net: LED15.2 (DOUT), LED16.3 (DIN)
- new net: LED12.2 (DOUT), LED13.3 (DIN)
- new net: LED11.2 (DOUT), LED12.3 (DIN)
- new net: LED4.2 (DOUT), LED7.3 (DIN)
- new net: LED3.2 (DOUT), LED4.3 (DIN)
- new net: LED1.2 (DOUT), LED2.3 (DIN)
- new net: LED10.2 (DOUT), LED11.3 (DIN)
- new net: LED3.3 (DIN), LED6.2 (DOUT)
- new net: LED10.3 (DIN), LED9.2 (DOUT)
- new net: LED5.2 (DOUT), LED6.3 (DIN)
- new net: LED2.2 (DOUT), LED5.3 (DIN)
- new net: LED8.2 (DOUT), LED9.3 (DIN)
- new net: LED14.2 (DOUT), LED15.3 (DIN)
- new net: LED7.2 (DOUT), LED8.3 (DIN)
- new net: LED13.2 (DOUT), LED14.3 (DIN)
- new net: LED19.2 (DOUT), LED20.3 (DIN)
- new net D_P: R4.1, U4.1 (I/O1)
- new net LED_5_data: LED1.3 (DIN), U6.4 (B)
- no-connect marks 2 -> 15
Other:
- note added: "1k resistor to not overdrive the crystal"
- note added: "Capacitors should have C0G dialectric to minimize DC bias."
- note added: "LEDs and decoupling capacitors"
- note added: "Level shifting"
- note added: "MAKE SURE TO SWAP THE TX AND RX PIN ON THE OTHER BOARD"
- note added: "MCU and decoupling"
- note added: "NOR FLASH"
- note added: "QUARTZ CRYSTAL"
- note added: "Switch matrix"
- note added: "USB C Power and ESD"
- note added: "USB C Split Connection and ESD"
- note removed: "The return path has to be very short under the chip or ground plane"
- moved on the sheet: C10, C11, C12, C13, C14, C15, C3, C4, C5, C6, C7, C8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

Commit message: started keyboard rounting
Parts:
- renumbered C22 to C20, C23 to C21, C20 to C22, C21 to C23, LED5 to LED3, LED6 to LED4, LED3 to LED5, LED4 to LED6
Connections:
- net LED_5_data: now also LED6.3 (DIN); no longer LED1.3 (DIN)
- net VBUS: now reaches D1.2 (A), J1.A4 (VBUS), J1.A9 (VBUS), J1.B4 (VBUS), J1.B9 (VBUS)
- net LED17IN: now reaches LED18.2 (DOUT)
- net LED17IN: now also LED17.3 (DIN); no longer LED19.3 (DIN)
- net LED16IN: now reaches LED17.2 (DOUT)
- net LED16IN: now also LED16.3 (DIN); no longer LED18.3 (DIN)
- net LED21IN: now reaches LED20.2 (DOUT), LED21.3 (DIN)
- net LED15IN: now reaches LED16.2 (DOUT)
- net LED15IN: now also LED15.3 (DIN); no longer LED17.3 (DIN)
- net CC1: now reaches J1.A5 (CC1), R1.1
- net LED14IN: now reaches LED15.2 (DOUT)
- net LED14IN: now also LED14.3 (DIN); no longer LED16.3 (DIN)
- net LED13IN: now reaches LED13.3 (DIN)
- net LED13IN: now also LED14.2 (DOUT); no longer LED12.2 (DOUT)
- net LED12IN: now reaches LED11.2 (DOUT), LED12.3 (DIN)
- net LED5IN: now reaches LED6.2 (DOUT)
- net LED5IN: now also LED5.3 (DIN); no longer LED7.3 (DIN)
- net LED4IN: now reaches LED5.2 (DOUT)
- net LED4IN: now also LED4.3 (DIN); no longer LED6.3 (DIN)
- net LED2IN: now reaches LED2.3 (DIN)
- net LED2IN: now also LED3.2 (DOUT); no longer LED1.2 (DOUT)
- net LED11IN: now reaches LED10.2 (DOUT), LED11.3 (DIN)
- net LED3IN: now reaches LED4.2 (DOUT)
- net LED3IN: now also LED3.3 (DIN); no longer LED5.3 (DIN)
- net CC2: now reaches J1.B5 (CC2), R2.1
- net LED10IN: now reaches LED10.3 (DIN), LED9.2 (DOUT)
- net LED1IN: now reaches LED2.2 (DOUT)
- net LED1IN: now also LED1.3 (DIN); no longer LED3.3 (DIN)
- net LED9IN: now reaches LED8.2 (DOUT), LED9.3 (DIN)
- net LED8IN: now reaches LED7.2 (DOUT), LED8.3 (DIN)
- net LED19IN: now reaches LED13.2 (DOUT)
- net LED19IN: now also LED19.3 (DIN); no longer LED14.3 (DIN)
- net LED20IN: now reaches LED19.2 (DOUT), LED20.3 (DIN)
- new net LED18IN: LED12.2 (DOUT), LED18.3 (DIN)
- new net LED7IN: LED1.2 (DOUT), LED7.3 (DIN)
Other:
- moved on the sheet: D1, R1, R2

Commit message: finished pcb layout
Parts:
- removed D1: SS34, Diode_SMD:D_SMA, symbol Diode:SS34
- added C79, C80: 100n, Capacitor_SMD:C_0402_1005Metric, symbol Device:C
- added D1: SS14, Diode_SMD:D_SMA, symbol Diode:SS14
Connections:
- net +3V3: now also C80.1
- net +5V: now also C79.1, D1.1 (K)
- net D_N: now also R4.1; no longer R3.1
- net D_P: now also R3.1; no longer R4.1
- net GND: now also C79.2, C80.2
- net SW1: now also U1.31 (GPIO20); no longer U1.7 (GPIO5)
- net SW10: now also U1.30 (GPIO19); no longer U1.17 (GPIO14)
- net SW11: now also U1.16 (GPIO13); no longer U1.18 (GPIO15)
- net SW12: now also U1.15 (GPIO12); no longer U1.27 (GPIO16)
- net SW13: now also U1.11 (GPIO8); no longer U1.28 (GPIO17)
- net SW14: now also U1.12 (GPIO9); no longer U1.29 (GPIO18)
- net SW15: now also U1.13 (GPIO10); no longer U1.30 (GPIO19)
- net SW16: now also U1.14 (GPIO11); no longer U1.31 (GPIO20)
- net SW17: now also U1.9 (GPIO7); no longer U1.32 (GPIO21)
- net SW18: now also U1.8 (GPIO6); no longer U1.34 (GPIO22)
- net SW19: now also U1.7 (GPIO5); no longer U1.35 (GPIO23)
- net SW2: now also U1.37 (GPIO25); no longer U1.8 (GPIO6)
- net SW20: now also U1.6 (GPIO4); no longer U1.36 (GPIO24)
- net SW21: now also U1.5 (GPIO3); no longer U1.37 (GPIO25)
- net SW3: now also U1.36 (GPIO24); no longer U1.9 (GPIO7)
- net SW4: now also U1.35 (GPIO23); no longer U1.11 (GPIO8)
- net SW5: now also U1.34 (GPIO22); no longer U1.12 (GPIO9)
- net SW6: now also U1.32 (GPIO21); no longer U1.13 (GPIO10)
- net SW7: now also U1.27 (GPIO16); no longer U1.14 (GPIO11)
- net SW8: now also U1.28 (GPIO17); no longer U1.15 (GPIO12)
- net SW9: now also U1.29 (GPIO18); no longer U1.16 (GPIO13)
- net VBUS: now also D1.2 (A)
- net DIR3V3: now reaches R8.1, U6.5 (DIR)
- net NCS: now reaches R6.1, SW98.1
- net TX_IN: now reaches J2.A7 (D-), J2.B7 (D-), U5.1 (I/O1)
- net RX_IN: now reaches J2.A6 (D+), J2.B6 (D+), U5.3 (I/O2)
- net CLimit: now reaches C16.1, R7.2, Y1.1
- net USB_DN: now reaches R4.2, U1.46 (USB_DM)
- net USB_DP: now reaches R3.2, U1.47 (USB_DP)
Other:
- moved on the sheet: R3, R4, R7, R8
