File: PCB/EagleV1/RightSide.kicad_sch (KiCad schematic)
At the start: 0 parts

Commit message: finished schematic
Parts:
- added C40, C41, C43, C44, C46, C48, C50, C51, C53, C54, C56, C57, C58, C59, C60, C61, C62, C63, C64, C65, C66, C67, C68, C69, C70, C71, C72, C73, C74, C75, C76, C77, C78: 100n, Capacitor_SMD:C_0402_1005Metric, symbol Device:C
- added C42, C45, C47, C49: 1u, Capacitor_SMD:C_0603_1608Metric, symbol Device:C
- added C52, C55: 15p, Capacitor_SMD:C_0402_1005Metric, symbol Device:C
- added D2: SS34, Diode_SMD:D_SMA, symbol Diode:SS34
- added J3, J4: USB_C_Receptacle_USB2.0_16P, Connector_USB:USB_C_Receptacle_G-Switch_GT-USB-7010ASV, symbol Connector:USB_C_Receptacle_USB2.0_16P
- added LED22, LED23, LED24, LED25, LED26, LED27, LED28, LED29, LED30, LED31, LED32, LED33, LED34, LED35, LED36, LED37, LED38, LED39, LED40, LED41, LED42: SK6812MINI-E, PCM_marbastlib-various:LED_6028R, symbol PCM_marbastlib-various:SK6812MINI-E
- added R10, R11: 27, Resistor_SMD:R_0402_1005Metric, symbol Device:R
- added R12, R16: 10k, Resistor_SMD:R_0402_1005Metric, symbol Device:R
- added R13, R14: 5.1k, Resistor_SMD:R_0402_1005Metric, symbol Device:R
- added R15, R9: 1k, Resistor_SMD:R_0402_1005Metric, symbol Device:R
- added SW22, SW23, SW24, SW25, SW26, SW27, SW28, SW29, SW30, SW31, SW32, SW33, SW34, SW35, SW36, SW37, SW38, SW39, SW40, SW41, SW42: SW_Push, RandomStuff4Keebs:SW_Redragon_LowProfile_PCB_1.00u, symbol Switch:SW_Push
- added SW99: TS-1088-AR02016, XUNPU TS-1088-AR02016:SW_TS-1088_XNP, symbol XUNPU TS-1088-AR02016:TS-1088-AR02016
- added U10: TLV1117-33, Package_TO_SOT_SMD:SOT-223-3_TabPin2, symbol Regulator_Linear:TLV1117-33
- added U11, U8: USBLC6-2SC6, Package_TO_SOT_SMD:SOT-23-6, symbol Power_Protection:USBLC6-2SC6
- added U12: SN74LVC1T45DCK, Package_TO_SOT_SMD:SOT-363_SC-70-6, symbol Logic_LevelTranslator:SN74LVC1T45DCK
- added U7: W25Q128JVS, Package_SO:SOIC-8_5.23x5.23mm_P1.27mm, symbol Memory_Flash:W25Q128JVS
- added U9: RP2040, Package_DFN_QFN:QFN-56-1EP_7x7mm_P0.4mm_EP3.2x3.2mm, symbol MCU_RaspberryPi:RP2040
- added Y2: Crystal_GNDB24, Crystal:Crystal_SMD_3225-4Pin_3.2x2.5mm, symbol Device:Crystal_GND24
Connections:
- new net: C52.1, R15.2, Y2.1
- new net: R9.1, SW99.1
- new net: LED38.2 (DOUT), LED42.3 (DIN)
- new net: LED28.2 (DOUT), LED31.3 (DIN)
- new net: LED25.2 (DOUT), LED28.3 (DIN)
- new net: LED33.2 (DOUT), LED37.3 (DIN)
- new net: LED30.2 (DOUT), LED33.3 (DIN)
- new net: J3.A5 (CC1), R13.1
- new net: LED24.3 (DIN), LED40.2 (DOUT)
- new net: LED36.2 (DOUT), LED40.3 (DIN)
- new net: LED22.2 (DOUT), LED25.3 (DIN)
- new net: LED37.2 (DOUT), LED41.3 (DIN)
- new net: R11.2, U9.46 (USB_DM)
- new net: LED26.2 (DOUT), LED29.3 (DIN)
- new net: LED23.2 (DOUT), LED26.3 (DIN)
- new net: LED24.2 (DOUT), LED27.3 (DIN)
- new net: LED32.2 (DOUT), LED36.3 (DIN)
- new net: LED29.2 (DOUT), LED32.3 (DIN)
- new net: R10.2, U9.47 (USB_DP)
- new net: LED23.3 (DIN), LED39.2 (DOUT)
- new net: R16.1, U12.5 (DIR)
- new net: LED34.2 (DOUT), LED38.3 (DIN)
- new net: LED27.2 (DOUT), LED30.3 (DIN)
- new net: D2.2 (A), J3.A4 (VBUS), J3.A9 (VBUS), J3.B4 (VBUS), J3.B9 (VBUS)
- new net: J3.B5 (CC2), R14.1
- new net: LED34.3 (DIN), LED41.2 (DOUT)
- new net: LED35.2 (DOUT), LED39.3 (DIN)
- new net: J4.A7 (D-), J4.B7 (D-), U8.1 (I/O1)
- new net: J4.A6 (D+), J4.B6 (D+), U8.3 (I/O2)
- new net: LED31.2 (DOUT), LED35.3 (DIN)
- new net +1V1B: C40.1, C41.1, C42.1, U9.23 (DVDD), U9.45 (VREG_VOUT), U9.50 (DVDD)
- new net +3V3B: C44.1, C47.1, C48.1, C49.1, C50.1, C51.1, C53.1, C54.1, C56.1, C57.1, R12.2, R16.2, U10.2 (VO), U12.1 (VCCA), U7.8 (VCC), U9.1 (IOVDD), U9.10 (IOVDD), U9.22 (IOVDD), U9.26 (RUN), U9.33 (IOVDD), U9.42 (IOVDD), U9.43 (ADC_AVDD), U9.44 (VREG_IN), U9.48 (USB_VDD), U9.49 (IOVDD)
- new net +5VB: C43.2, C45.1, C46.2, C58.2, C59.2, C60.2, C61.2, C62.2, C63.2, C64.2, C65.2, C66.2, C67.2, C68.2, C69.2, C70.2, C71.2, C72.2, C73.2, C74.2, C75.2, C76.2, C77.2, C78.2, D2.1 (K), J4.A4 (VBUS), J4.A9 (VBUS), J4.B4 (VBUS), J4.B9 (VBUS), LED22.1 (VDD), LED23.1 (VDD), LED24.1 (VDD), LED25.1 (VDD), LED26.1 (VDD), LED27.1 (VDD), LED28.1 (VDD), LED29.1 (VDD), LED30.1 (VDD), LED31.1 (VDD), LED32.1 (VDD), LED33.1 (VDD), LED34.1 (VDD), LED35.1 (VDD), LED36.1 (VDD), LED37.1 (VDD), LED38.1 (VDD), LED39.1 (VDD), LED40.1 (VDD), LED41.1 (VDD), LED42.1 (VDD), U10.3 (VI), U11.5 (VBUS), U12.6 (VCCB), U8.5 (VBUS)
- new net D+_B: J3.A6 (D+), J3.B6 (D+), U11.6 (I/O1)
- new net D-_B: J3.A7 (D-), J3.B7 (D-), U11.4 (I/O2)
- new net D_N_B: R10.1, U11.3 (I/O2)
- new net D_P_B: R11.1, U11.1 (I/O1)
- new net GNDB: C40.2, C41.2, C42.2, C43.1, C44.2, C45.2, C46.1, C47.2, C48.2, C49.2, C50.2, C51.2, C52.2, C53.2, C54.2, C55.2, C56.2, C57.2, C58.1, C59.1, C60.1, C61.1, C62.1, C63.1, C64.1, C65.1, C66.1, C67.1, C68.1, C69.1, C70.1, C71.1, C72.1, C73.1, C74.1, C75.1, C76.1, C77.1, C78.1, J3.A1 (GND), J3.A12 (GND), J3.B1 (GND), J3.B12 (GND), J3.S1 (SHIELD), J4.A1 (GND), J4.A12 (GND), J4.B1 (GND), J4.B12 (GND), J4.S1 (SHIELD), LED22.4 (VSS), LED23.4 (VSS), LED24.4 (VSS), LED25.4 (VSS), LED26.4 (VSS), LED27.4 (VSS), LED28.4 (VSS), LED29.4 (VSS), LED30.4 (VSS), LED31.4 (VSS), LED32.4 (VSS), LED33.4 (VSS), LED34.4 (VSS), LED35.4 (VSS), LED36.4 (VSS), LED37.4 (VSS), LED38.4 (VSS), LED39.4 (VSS), LED40.4 (VSS), LED41.4 (VSS), LED42.4 (VSS), R13.2, R14.2, SW22.2, SW23.2, SW24.2, SW25.2, SW26.2, SW27.2, SW28.2, SW29.2, SW30.2, SW31.2, SW32.2, SW33.2, SW34.2, SW35.2, SW36.2, SW37.2, SW38.2, SW39.2, SW40.2, SW41.2, SW42.2, SW99.2, U10.1 (GND), U11.2 (GND), U12.2 (GND), U7.4 (GND), U8.2 (GND), U9.19 (TESTEN), U9.57 (GND), Y2.2, Y2.4
- new net LED_33_data_B: U12.3 (A), U9.4 (GPIO2)
- new net LED_5_data_B: LED22.3 (DIN), U12.4 (B)
- new net QSPI_CLK: U7.6 (CLK), U9.52 (QSPI_SCLK)
- new net QSPI_D0: U7.5 (DI(IO0)), U9.53 (QSPI_SD0)
- new net QSPI_D1: U7.2 (DO(IO1)), U9.55 (QSPI_SD1)
- new net QSPI_D2: U7.3 (IO2), U9.54 (QSPI_SD2)
- new net QSPI_D3: U7.7 (IO3), U9.51 (QSPI_SD3)
- new net QSPI_NCS: R12.1, R9.2, U7.1 (~{CS}), U9.56 (QSPI_SS)
- new net RXB: U8.4 (I/O2), U9.2 (GPIO0)
- new net SW22: SW22.1, U9.7 (GPIO5)
- new net SW23: SW23.1, U9.8 (GPIO6)
- new net SW24: SW24.1, U9.9 (GPIO7)
- new net SW25: SW25.1, U9.11 (GPIO8)
- new net SW26: SW26.1, U9.12 (GPIO9)
- new net SW27: SW27.1, U9.13 (GPIO10)
- new net SW28: SW28.1, U9.14 (GPIO11)
- new net SW29: SW29.1, U9.15 (GPIO12)
- new net SW30: SW30.1, U9.16 (GPIO13)
- new net SW31: SW31.1, U9.17 (GPIO14)
- new net SW32: SW32.1, U9.18 (GPIO15)
- new net SW33: SW33.1, U9.27 (GPIO16)
- new net SW34: SW34.1, U9.28 (GPIO17)
- new net SW35: SW35.1, U9.29 (GPIO18)
- new net SW36: SW36.1, U9.30 (GPIO19)
- new net SW37: SW37.1, U9.31 (GPIO20)
- new net SW38: SW38.1, U9.32 (GPIO21)
- new net SW39: SW39.1, U9.34 (GPIO22)
- new net SW40: SW40.1, U9.35 (GPIO23)
- new net SW41: SW41.1, U9.36 (GPIO24)
- new net SW42: SW42.1, U9.37 (GPIO25)
- new net TXB: U8.6 (I/O1), U9.3 (GPIO1)
- new net XINB: C55.1, U9.20 (XIN), Y2.3
- new net XOUTB: R15.1, U9.21 (XOUT)
- no-connect marks 0 -> 15
Other:
- note added: "1k resistor to not overdrive the crystal"
- note added: "Capacitors should have C0G dialectric to minimize DC bias."
- note added: "LEDs and decoupling capacitors"
- note added: "Level shifting"
- note added: "MAKE SURE TO SWAP THE TXB AND RXB PIN ON THE OTHER BOARD"
- note added: "MCU and decoupling"
- note added: "NOR FLASH"
- note added: "QUARTZ CRYSTAL"
- note added: "Switch matrix"
- note added: "USB C Power and ESD"
- note added: "USB C Split Connection and ESD"

Commit message: started keyboard rounting
Parts:
- renumbered C61 to C59, C64 to C60, C67 to C61, C71 to C62, C75 to C63, C59 to C64, C62 to C65, C65 to C66, C68 to C67, C72 to C68, C76 to C69, C60 to C70, C63 to C71, C66 to C72, C69 to C73, C73 to C74, C77 to C75, C70 to C76, C74 to C77, LED25 to LED23, LED28 to LED24, LED31 to LED25, LED35 to LED26, LED39 to LED27, LED23 to LED28, LED26 to LED29, LED29 to LED30, LED32 to LED31, LED36 to LED32, LED40 to LED33, LED24 to LED34, LED27 to LED35, LED30 to LED36, LED33 to LED37, LED37 to LED38, LED41 to LED39, LED34 to LED40, LED38 to LED41
Connections:
- net CC1B: now reaches J3.A5 (CC1), R13.1
- net VBUSB: now reaches D2.2 (A), J3.A4 (VBUS), J3.A9 (VBUS), J3.B4 (VBUS), J3.B9 (VBUS)
- net CC2B: now reaches J3.B5 (CC2), R14.1
- net QSPI_CLK renamed QSPI_CLK_B
- net QSPI_D0 renamed QSPI_D0_B
- net QSPI_D1 renamed QSPI_D1_B
- net QSPI_D2 renamed QSPI_D2_B
- net QSPI_D3 renamed QSPI_D3_B
- net QSPI_NCS renamed QSPI_NCS_B_B
- net QSPI_NCS_B_B: no longer U9.56 (QSPI_SS)
- new net QSPI_NCS_B: U9.56 (QSPI_SS)
Other:
- moved on the sheet: D2, R13, R14

Commit message: finished pcb layout
Parts:
- removed D2: SS34, Diode_SMD:D_SMA, symbol Diode:SS34
- added C81, C82: 100n, Capacitor_SMD:C_0402_1005Metric, symbol Device:C
- added D2: SS14, Diode_SMD:D_SMA, symbol Diode:SS14
Connections:
- net +3V3B: now also C82.1
- net +5VB: now also C81.1, D2.1 (K)
- net D_N_B: now also R11.1; no longer R10.1
- net D_P_B: now also R10.1; no longer R11.1
- net SW22: no longer U9.7 (GPIO5)
- net SW23: no longer U9.8 (GPIO6)
- net SW24: no longer U9.9 (GPIO7)
- net SW25: no longer U9.11 (GPIO8)
- net SW26: no longer U9.12 (GPIO9)
- net SW27: no longer U9.13 (GPIO10)
- net SW28: no longer U9.14 (GPIO11)
- net SW29: no longer U9.15 (GPIO12)
- net SW30: no longer U9.16 (GPIO13)
- net SW31: no longer U9.17 (GPIO14)
- net SW32: no longer U9.18 (GPIO15)
- net SW33: no longer U9.27 (GPIO16)
- net SW34: no longer U9.28 (GPIO17)
- net SW35: no longer U9.29 (GPIO18)
- net SW36: no longer U9.30 (GPIO19)
- net SW37: no longer U9.31 (GPIO20)
- net SW38: no longer U9.32 (GPIO21)
- net SW39: no longer U9.34 (GPIO22)
- net SW40: no longer U9.35 (GPIO23)
- net SW41: no longer U9.36 (GPIO24)
- net SW42: no longer U9.37 (GPIO25)
- net VBUSB: now also D2.2 (A)
- net CLimitB: now reaches C52.1, R15.2, Y2.1
- net USBB_DN: now reaches R11.2, U9.46 (USB_DM)
- net USBB_DP: now reaches R10.2, U9.47 (USB_DP)
- net DIR3V3B: now reaches R16.1, U12.5 (DIR)
- net TXB_IN: now reaches J4.A7 (D-), J4.B7 (D-), U8.1 (I/O1)
- net RXB_IN: now reaches J4.A6 (D+), J4.B6 (D+), U8.3 (I/O2)
- new net GND: C81.2, C82.2
Other:
- moved on the sheet: R10, R11, R15, R16

Commit message: routed all the tracks and smds
Connections:
- net QSPI_NCS_B_B is gone; now on net QSPI_NCS_B: R12.1, R9.2, U7.1 (~{CS})
- net +5VB: no longer C58.2, C59.2, C60.2, C61.2, C62.2, C63.2, C64.2, C65.2, C66.2, C67.2, C68.2, C69.2, C70.2, C71.2, C72.2, C73.2, C74.2, C75.2, C76.2, C77.2, C78.2, LED22.1 (VDD), LED23.1 (VDD), LED24.1 (VDD), LED25.1 (VDD), LED26.1 (VDD), LED27.1 (VDD), LED28.1 (VDD), LED29.1 (VDD), LED30.1 (VDD), LED31.1 (VDD), LED32.1 (VDD), LED33.1 (VDD), LED34.1 (VDD), LED35.1 (VDD), LED36.1 (VDD), LED37.1 (VDD), LED38.1 (VDD), LED39.1 (VDD), LED40.1 (VDD), LED41.1 (VDD), LED42.1 (VDD)
- net GND: now also C58.1, C59.1, C60.1, C61.1, C62.1, C63.1, C64.1, C65.1, C66.1, C67.1, C68.1, C69.1, C70.1, C71.1, C72.1, C73.1, C74.1, C75.1, C76.1, C77.1, C78.1, LED22.4 (VSS), LED23.4 (VSS), LED24.4 (VSS), LED25.4 (VSS), LED26.4 (VSS), LED27.4 (VSS), LED28.4 (VSS), LED29.4 (VSS), LED30.4 (VSS), LED31.4 (VSS), LED32.4 (VSS), LED33.4 (VSS), LED34.4 (VSS), LED35.4 (VSS), LED36.4 (VSS), LED37.4 (VSS), LED38.4 (VSS), LED39.4 (VSS), LED40.4 (VSS), LED41.4 (VSS), LED42.4 (VSS)
- net GNDB: no longer C58.1, C59.1, C60.1, C61.1, C62.1, C63.1, C64.1, C65.1, C66.1, C67.1, C68.1, C69.1, C70.1, C71.1, C72.1, C73.1, C74.1, C75.1, C76.1, C77.1, C78.1, LED22.4 (VSS), LED23.4 (VSS), LED24.4 (VSS), LED25.4 (VSS), LED26.4 (VSS), LED27.4 (VSS), LED28.4 (VSS), LED29.4 (VSS), LED30.4 (VSS), LED31.4 (VSS), LED32.4 (VSS), LED33.4 (VSS), LED34.4 (VSS), LED35.4 (VSS), LED36.4 (VSS), LED37.4 (VSS), LED38.4 (VSS), LED39.4 (VSS), LED40.4 (VSS), LED41.4 (VSS), LED42.4 (VSS)
- net SW22: now also U9.5 (GPIO3)
- net SW23: now also U9.6 (GPIO4)
- net SW24: now also U9.7 (GPIO5)
- net SW25: now also U9.8 (GPIO6)
- net SW26: now also U9.9 (GPIO7)
- net SW27: now also U9.11 (GPIO8)
- net SW28: now also U9.12 (GPIO9)
- net SW29: now also U9.13 (GPIO10)
- net SW30: now also U9.14 (GPIO11)
- net SW31: now also U9.15 (GPIO12)
- net SW32: now also U9.16 (GPIO13)
- net SW33: now also U9.17 (GPIO14)
- net SW34: now also U9.27 (GPIO16)
- net SW35: now also U9.28 (GPIO17)
- net SW36: now also U9.29 (GPIO18)
- net SW37: now also U9.30 (GPIO19)
- net SW38: now also U9.31 (GPIO20)
- net SW39: now also U9.32 (GPIO21)
- net SW40: now also U9.36 (GPIO24)
- net SW41: now also U9.35 (GPIO23)
- net SW42: now also U9.34 (GPIO22)
- net NCSB: now reaches R9.1, SW99.1
- net LED41IN: now reaches LED42.2 (DOUT)
- net LED41IN: now also LED41.3 (DIN)
- net LED40IN: now reaches LED41.2 (DOUT)
- net LED40IN: now also LED40.3 (DIN); no longer LED42.3 (DIN)
- net LED25IN: now reaches LED24.2 (DOUT), LED25.3 (DIN)
- net LED24IN: now reaches LED23.2 (DOUT), LED24.3 (DIN)
- net LED38IN: now reaches LED37.2 (DOUT), LED38.3 (DIN)
- net LED37IN: now reaches LED36.2 (DOUT), LED37.3 (DIN)
- net LED32IN: now reaches LED33.2 (DOUT)
- net LED32IN: now also LED32.3 (DIN); no longer LED34.3 (DIN)
- net LED31IN: now reaches LED32.2 (DOUT)
- net LED31IN: now also LED31.3 (DIN); no longer LED33.3 (DIN)
- net LED23IN: now reaches LED22.2 (DOUT), LED23.3 (DIN)
- net LED39IN: now reaches LED38.2 (DOUT), LED39.3 (DIN)
- net LED28IN: now reaches LED29.2 (DOUT)
- net LED28IN: now also LED28.3 (DIN); no longer LED30.3 (DIN)
- net LED29IN: now reaches LED29.3 (DIN)
- net LED29IN: now also LED30.2 (DOUT); no longer LED28.2 (DOUT)
- net LED35IN: now reaches LED34.2 (DOUT), LED35.3 (DIN)
- net LED30IN: now reaches LED31.2 (DOUT)
- net LED30IN: now also LED30.3 (DIN); no longer LED32.3 (DIN)
- net LED33IN: now reaches LED27.2 (DOUT)
- net LED33IN: now also LED33.3 (DIN); no longer LED28.3 (DIN)
- net at LED40.2 (DOUT): no longer LED41.3 (DIN)
- net LED36IN: now reaches LED35.2 (DOUT), LED36.3 (DIN)
- net LED42IN: now reaches LED39.2 (DOUT)
- net LED42IN: now also LED42.3 (DIN); no longer LED40.3 (DIN)
- net LED27IN: now reaches LED26.2 (DOUT), LED27.3 (DIN)
- net LED26IN: now reaches LED25.2 (DOUT), LED26.3 (DIN)
- new net +5V: C58.2, C59.2, C60.2, C61.2, C62.2, C63.2, C64.2, C65.2, C66.2, C67.2, C68.2, C69.2, C70.2, C71.2, C72.2, C73.2, C74.2, C75.2, C76.2, C77.2, C78.2, LED22.1 (VDD), LED23.1 (VDD), LED24.1 (VDD), LED25.1 (VDD), LED26.1 (VDD), LED27.1 (VDD), LED28.1 (VDD), LED29.1 (VDD), LED30.1 (VDD), LED31.1 (VDD), LED32.1 (VDD), LED33.1 (VDD), LED34.1 (VDD), LED35.1 (VDD), LED36.1 (VDD), LED37.1 (VDD), LED38.1 (VDD), LED39.1 (VDD), LED40.1 (VDD), LED41.1 (VDD), LED42.1 (VDD)
- new net LED34IN: LED28.2 (DOUT), LED34.3 (DIN)

Commit message: Finished layout, both halves
Connections:
- net +5V is gone; now on net +5VB: C58.2, C59.2, C60.2, C61.2, C62.2, C63.2, C64.2, C65.2, C66.2, C67.2, C68.2, C69.2, C70.2, C71.2, C72.2, C73.2, C74.2, C75.2, C76.2, C77.2, C78.2, LED22.1 (VDD), LED23.1 (VDD), LED24.1 (VDD), LED25.1 (VDD), LED26.1 (VDD), LED27.1 (VDD), LED28.1 (VDD), LED29.1 (VDD), LED30.1 (VDD), LED31.1 (VDD), LED32.1 (VDD), LED33.1 (VDD), LED34.1 (VDD), LED35.1 (VDD), LED36.1 (VDD), LED37.1 (VDD), LED38.1 (VDD), LED39.1 (VDD), LED40.1 (VDD), LED41.1 (VDD), LED42.1 (VDD)
- net GND is gone; now on net GNDB: C58.1, C59.1, C60.1, C61.1, C62.1, C63.1, C64.1, C65.1, C66.1, C67.1, C68.1, C69.1, C70.1, C71.1, C72.1, C73.1, C74.1, C75.1, C76.1, C77.1, C78.1, C81.2, C82.2, LED22.4 (VSS), LED23.4 (VSS), LED24.4 (VSS), LED25.4 (VSS), LED26.4 (VSS), LED27.4 (VSS), LED28.4 (VSS), LED29.4 (VSS), LED30.4 (VSS), LED31.4 (VSS), LED32.4 (VSS), LED33.4 (VSS), LED34.4 (VSS), LED35.4 (VSS), LED36.4 (VSS), LED37.4 (VSS), LED38.4 (VSS), LED39.4 (VSS), LED40.4 (VSS), LED41.4 (VSS), LED42.4 (VSS)
Changed lines of the file:
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@@
 			)
 		)
-		(property "Value" "GND"
+		(property "Value" "GNDB"
 			(at 193.802 108.458 0)
 			(effects
@@
 			)
 		)
-		(property "Value" "GND"
+		(property "Value" "GNDB"
 			(at 171.704 108.204 0)
 			(effects
@@
 			)
 		)
-		(property "Value" "+5V"
+		(property "Value" "+5VB"
 			(at 345.44 20.32 0)
 			(effects
@@
 			)
 		)
-		(property "Value" "GND"
+		(property "Value" "GNDB"
 			(at 339.09 152.4 0)
 			(effects
